File: A1200PcmciaResetFix/A1200PcmciaResetFix.kicad_pcb (KiCad board)
At the start: 2 copper layers, 40 x 35.6 mm, 7 parts, among them J1 ADDR, J2 RESET, Q1 BC807, U1 ACT1225PL84

Commit message: A1200PcmciaResetFix, A600-1200KeyboardSocket : update socket symbol and footprint, no PCB change
Parts:
- removed U1: ACT1225PL84, Package_LCC:PLCC-84_THT-Socket
- added U5: GAYLE, Sassa:PLCC-84_THT-SocketOnTop, B.Cu at (114.3, 83.8)
